File: CapacitorSuperChargeCircuit.kicad_sch (KiCad schematic)
At the start: 19 parts, among them J2 Screw_Terminal_01x02, J3 Screw_Terminal_01x02, U1 PAM2421AECADJR

Commit message: v2 smd version foxed
Parts:
- removed C2, C4: 10uF, Capacitor_THT:CP_Radial_D5.0mm_P2.50mm, symbol Device:C_Polarized
- removed U1: PAM2421AECADJR, Package_SO:Infineon_PG-DSO-8-43, symbol Connector:Conn_01x09_Pin
- added C2, C4: 10μF 16V X5R, Capacitor_SMD:C_0603_1608Metric_Pad1.08x0.95mm_HandSolder, symbol Device:C
- added U1: ~, Library:PAM242x, symbol New_Library:PAM242x
- C1, C5: value 470uF -> 16V 470uF; footprint Capacitor_THT:CP_Radial_D6.3mm_P2.50mm -> Capacitor_THT:CP_Radial_D8.0mm_P3.50mm
- C3, C9: value 1uF -> 1μF 25V X7R; footprint Capacitor_THT:C_Disc_D3.4mm_W2.1mm_P2.50mm -> Capacitor_SMD:C_0603_1608Metric_Pad1.08x0.95mm_HandSolder
- C6: value 47pF -> 47pF 50V CH; footprint Capacitor_THT:C_Disc_D3.4mm_W2.1mm_P2.50mm -> Capacitor_SMD:C_0603_1608Metric_Pad1.08x0.95mm_HandSolder
- C7: value 2.2nF -> 2.2nF 50V X7R; footprint Capacitor_THT:C_Disc_D3.4mm_W2.1mm_P2.50mm -> Capacitor_SMD:C_0603_1608Metric_Pad1.08x0.95mm_HandSolder
- C8: value 10nF -> 0.47μF 50V X7R; footprint Capacitor_THT:C_Disc_D3.4mm_W2.1mm_P2.50mm -> Capacitor_SMD:C_0603_1608Metric_Pad1.08x0.95mm_HandSolder
- D1: value D_Schottky -> RB160M-30TR; footprint Diode_THT:D_A-405_P7.62mm_Horizontal -> Diode_SMD:D_SOD-123
- FB1, FB2: value FerriteBead -> BLM18PG471SN1D; footprint Inductor_THT:L_Axial_L5.3mm_D2.2mm_P10.16mm_Horizontal_Vishay_IM-1 -> Inductor_SMD:L_0603_1608Metric
- L1: value AL0307-6R8K 6.8uH -> DFE322512F-100M; footprint Inductor_THT:L_Axial_L5.3mm_D2.2mm_P7.62mm_Horizontal_Vishay_IM-1 -> Inductor_SMD:L_1210_3225Metric_Pad1.42x2.65mm_HandSolder
- R1: value 85k -> 110k; footprint Resistor_THT:R_Axial_DIN0204_L3.6mm_D1.6mm_P7.62mm_Horizontal -> Resistor_SMD:R_0603_1608Metric_Pad0.98x0.95mm_HandSolder
- R2: value 10k -> 13k; footprint Resistor_THT:R_Axial_DIN0204_L3.6mm_D1.6mm_P7.62mm_Horizontal -> Resistor_SMD:R_0603_1608Metric_Pad0.98x0.95mm_HandSolder
- R3: footprint Resistor_THT:R_Axial_DIN0204_L3.6mm_D1.6mm_P7.62mm_Horizontal -> Resistor_SMD:R_0603_1608Metric_Pad0.98x0.95mm_HandSolder
Connections:
- net COMP: now also U1.4 (COMP)
- net FB: now also U1.6 (FB)
- net GND: now also C2.2, C4.2, U1.1 (PGND), U1.5 (AGND), U1.9 (PAD)
- net SS: now also U1.7 (SS)
- net SW: now also U1.8 (SW)
- net VIN: now also C2.1, U1.2 (VIN), U1.3 (EN)
- net VOUT: now also C4.1
Other:
- moved on the sheet: C1, C6, L1
